Commit message: fixed traj read real robot data

File: single_arm_6dof_description/urdf/single_arm_6dof.xacro (robot description, xacro)
@@ -13,15 +13,15 @@
     <inertial>
       <origin
-        xyz="-3.4663E-05 -4.5026E-05 0.0084004"
+        xyz="-0.00010098 -0.00035109 0.054127"
         rpy="0 0 0" />
       <mass
         value="2.94316" />
       <inertia
-        ixx="0.0094824"
+        ixx="0.00082016"
         ixy="3.555E-10"
         ixz="-4.1821E-06"
-        iyy="0.0095713"
-        iyz="-9.8398E-08"
-        izz="0.018031" />
+        iyy="0.00081979"
+        iyz="-1.4527E-07"
+        izz="0.00035328" />
     </inertial>
     <visual>
@@ -104,6 +104,6 @@
     type="revolute">
     <origin
-      xyz="0 -0.0685 0.0315"
-      rpy="1.5708 0 0" />
+      xyz="0 -0.0684999999999984 0.0315"
+      rpy="1.5707963267949 0 0" />
     <parent
       link="link1" />
@@ -121,15 +121,15 @@
     <inertial>
       <origin
-        xyz="-2.4369E-07 0.18004 0.0061614"
+        xyz="0.17471 2.0582E-07 0.0097884"
         rpy="0 0 0" />
       <mass
         value="1.07602" />
       <inertia
-        ixx="0.00076385"
-        ixy="2.1135E-12"
-        ixz="4.2672E-10"
-        iyy="0.00051784"
-        iyz="3.6733E-07"
-        izz="0.00050582" />
+        ixx="0.00054963"
+        ixy="-2.1133E-12"
+        ixz="3.6733E-07"
+        iyy="0.0010834"
+        iyz="-4.2672E-10"
+        izz="0.00082532" />
     </inertial>
     <visual>
@@ -161,6 +161,6 @@
     type="revolute">
     <origin
-      xyz="0 0.2675 -0.039"
-      rpy="-3.1416 0 3.1416" />
+      xyz="0.2675 0 -0.0390000000000001"
+      rpy="0 0 0" />
     <parent
       link="link2" />
@@ -168,4 +168,60 @@
       link="link3" />
     <axis
+      xyz="0 0 -1" />
+    <limit
+      lower="-3.14"
+      upper="3.14"
+      effort="0"
+      velocity="0" />
+  </joint>
+  <link name="link3">
+    <inertial>
+      <origin
+        xyz="0.14898 1.9084E-07 -0.006871"
+        rpy="0 0 0" />
+      <mass
+        value="1.00039" />
+      <inertia
+        ixx="0.00047701"
+        ixy="-1.0214E-11"
+        ixz="-1.2577E-06"
+        iyy="0.00077795"
+        iyz="-9.0438E-10"
+        izz="0.00054702" />
+    </inertial>
+    <visual>
+      <origin
+        xyz="0 0 0"
+        rpy="0 0 0" />
+      <geometry>
+        <mesh
+          filename="package://single_arm_6dof_description/meshes/link3.STL" />
+      </geometry>
+      <material
+        name="grey">
+        <color
+          rgba="0.792156862745098 0.819607843137255 0.933333333333333 1" />
+      </material>
+    </visual>
+    <collision>
+      <origin
+        xyz="0 0 0"
+        rpy="0 0 0" />
+      <geometry>
+        <mesh
+          filename="package://single_arm_6dof_description/meshes/link3.STL" />
+      </geometry>
+    </collision>
+  </link>
+  <joint name="joint4"
+    type="revolute">
+    <origin
+      xyz="0.2324 0 0.0390000000000069"
+      rpy="0 0 -3.14159265358979" />
+    <parent
+      link="link3" />
+    <child
+      link="link4" />
+    <axis
       xyz="0 0 1" />
     <limit
@@ -175,26 +231,26 @@
       velocity="0" />
   </joint>
-  <link name="link3">
-    <inertial>
-      <origin
-        xyz="2.2281E-07 0.15321 0.0030804"
-        rpy="0 0 0" />
-      <mass
-        value="1.00039" />
-      <inertia
-        ixx="0.00058978"
-        ixy="-1.0211E-11"
-        ixz="9.0438E-10"
-        iyy="0.000451"
-        iyz="1.2577E-06"
-        izz="0.00035885" />
-    </inertial>
-    <visual>
-      <origin
-        xyz="0 0 0"
-        rpy="0 0 0" />
-      <geometry>
-        <mesh
-          filename="package://single_arm_6dof_description/meshes/link3.STL" />
+  <link name="link4">
+    <inertial>
+      <origin
+        xyz="2.7756E-16 0.01039 0.02404"
+        rpy="0 0 0" />
+      <mass
+        value="0.36924" />
+      <inertia
+        ixx="9.4187E-05"
+        ixy="1.3079E-19"
+        ixz="-1.4502E-16"
+        iyy="4.476E-05"
+        iyz="5.3346E-07"
+        izz="0.0001027" />
+    </inertial>
+    <visual>
+      <origin
+        xyz="0 0 0"
+        rpy="0 0 0" />
+      <geometry>
+        <mesh
+          filename="package://single_arm_6dof_description/meshes/link4.STL" />
       </geometry>
       <material
@@ -210,75 +266,19 @@
       <geometry>
         <mesh
-          filename="package://single_arm_6dof_description/meshes/link3.STL" />
-      </geometry>
-    </collision>
-  </link>
-  <joint name="joint4"
-    type="revolute">
-    <origin
-      xyz="0 0.2324 -0.039"
-      rpy="-3.1416 0 1.5708" />
-    <parent
-      link="link3" />
-    <child
+          filename="package://single_arm_6dof_description/meshes/link4.STL" />
+      </geometry>
+    </collision>
+  </link>
+  <joint name="joint5"
+    type="revolute">
+    <origin
+      xyz="0 0.052 0.0286"
+      rpy="1.5707963267949 0 1.5707963267949" />
+    <parent
       link="link4" />
-    <axis
-      xyz="0 0 1" />
-    <limit
-      lower="-3.14"
-      upper="3.14"
-      effort="0"
-      velocity="0" />
-  </joint>
-  <link name="link4">
-    <inertial>
-      <origin
-        xyz="0.01039 -1.3878E-16 0.02404"
-        rpy="0 0 0" />
-      <mass
-        value="0.36924" />
-      <inertia
-        ixx="4.476E-05"
-        ixy="-1.095E-19"
-        ixz="5.3346E-07"
-        iyy="9.4187E-05"
-        iyz="1.4501E-16"
-        izz="0.0001027" />
-    </inertial>
-    <visual>
-      <origin
-        xyz="0 0 0"
-        rpy="0 0 0" />
-      <geometry>
-        <mesh
-          filename="package://single_arm_6dof_description/meshes/link4.STL" />
-      </geometry>
-      <material
-        name="grey">
-        <color
-          rgba="0.792156862745098 0.819607843137255 0.933333333333333 1" />
-      </material>
-    </visual>
-    <collision>
-      <origin
-        xyz="0 0 0"
-        rpy="0 0 0" />
-      <geometry>
-        <mesh
-          filename="package://single_arm_6dof_description/meshes/link4.STL" />
-      </geometry>
-    </collision>
-  </link>
-  <joint name="joint5"
-    type="revolute">
-    <origin
-      xyz="0.052 0 0.0286"
-      rpy="0 1.5708 0" />
-    <parent
-      link="link4" />
     <child
       link="link5" />
     <axis
-      xyz="0 0 1" />
+      xyz="1 0 0" />
     <limit
       lower="-3.14"
@@ -290,15 +290,15 @@
     <inertial>
       <origin
-        xyz="-0.010457 8.3267E-17 0.028614"
+        xyz="0.028614 0.010457 -1.6653E-16"
         rpy="0 0 0" />
       <mass
         value="0.36821" />
       <inertia
-        ixx="4.3878E-05"
-        ixy="-1.249E-19"
-        ixz="-5.3346E-07"
-        iyy="9.3658E-05"
-        iyz="-1.4501E-16"
-        izz="0.00010133" />
+        ixx="0.00010133"
+        ixy="5.3346E-07"
+        ixz="1.4501E-16"
+        iyy="4.3878E-05"
+        iyz="-9.098E-20"
+        izz="9.3658E-05" />
     </inertial>
     <visual>
@@ -330,6 +330,6 @@
     type="revolute">
     <origin
-      xyz="-0.055 0 0.033001"
-      rpy="0 -1.5708 0" />
+      xyz="0.0330005379381037 0.0549999394444907 0"
+      rpy="1.57079632679488 -1.5707963267949 0" />
     <parent
       link="link5" />
@@ -337,5 +337,5 @@
       link="link6" />
     <axis
-      xyz="0 0 1" />
+      xyz="0 0 -1" />
     <limit
       lower="-3.14"
@@ -347,15 +347,15 @@
     <inertial>
       <origin
-        xyz="-5.3794E-07 4.1633E-16 0.0070001"
-        rpy="0 0 0" />
-      <mass
-        value="0.025977" />
-      <inertia
-        ixx="2.2053E-06"
-        ixy="2.5014E-22"
-        ixz="-1.4272E-22"
-        iyy="2.2053E-06"
-        iyz="-1.2285E-22"
-        izz="3.9777E-06" />
+        xyz="-4.44089209850063E-16 5.37938091368581E-07 -0.00700006055550945"
+        rpy="0 0 0" />
+      <mass
+        value="0.0259770442543706" />
+      <inertia
+        ixx="2.20534281951167E-06"
+        ixy="1.78671012311437E-22"
+        ixz="-8.79317315621994E-22"
+        iyy="2.20534281951168E-06"
+        iyz="2.32583060538047E-20"
+        izz="3.9777349014505E-06" />
     </inertial>
     <visual>
