Commit message: save complex task structure

File: single_arm_6dof_description/urdf/single_arm_6dof.ros2_control.xacro (robot description, xacro)
@@ -7,5 +7,5 @@
         <param name="usb_port">/dev/ttyUSB0</param>
         <param name="baud_rate">115200</param>
-        <!-- <param name="use_dummy">true</param> -->
+        <param name="use_dummy">true</param>
       </hardware>
       <joint name="joint1">

File: single_arm_6dof_description/urdf/single_arm_6dof_simple.xacro (robot description, xacro)
@@ -121,15 +121,15 @@
     <inertial>
       <origin
-        xyz="0.18318 2.0418E-07 0.0099458"
-        rpy="0 0 0" />
-      <mass
-        value="1.2356" />
-      <inertia
-        ixx="0.00055193"
-        ixy="-2.1622E-12"
+        xyz="0.17471 2.0582E-07 0.0097884"
+        rpy="0 0 0" />
+      <mass
+        value="1.07602" />
+      <inertia
+        ixx="0.00054963"
+        ixy="-2.1133E-12"
         ixz="3.6733E-07"
-        iyy="0.0011981"
+        iyy="0.0010834"
         iyz="-4.2672E-10"
-        izz="0.00094005" />
+        izz="0.00082532" />
     </inertial>
     <visual>
@@ -161,5 +161,5 @@
     type="revolute">
     <origin
-      xyz="0.2819 0 -0.0390000000000005"
+      xyz="0.2675 0 -0.0390000000000001"
       rpy="0 0 0" />
     <parent
@@ -178,15 +178,15 @@
     <inertial>
       <origin
-        xyz="0.17413 1.7702E-07 -0.0085086"
-        rpy="0 0 0" />
-      <mass
-        value="1.1763" />
-      <inertia
-        ixx="0.00048947"
-        ixy="-1.0199E-11"
+        xyz="0.14898 1.9084E-07 -0.006871"
+        rpy="0 0 0" />
+      <mass
+        value="1.00039" />
+      <inertia
+        ixx="0.00047701"
+        ixy="-1.0214E-11"
         ixz="-1.2577E-06"
-        iyy="0.0011799"
+        iyy="0.00077795"
         iyz="-9.0438E-10"
-        izz="0.00094898" />
+        izz="0.00054702" />
     </inertial>
     <visual>
@@ -217,5 +217,5 @@
     type="revolute">
     <origin
-      xyz="0.278100000000002 0 0.0390000000000007"
+      xyz="0.2324 0 0.0390000000000069"
       rpy="0 0 -3.14159265358979" />
     <parent
@@ -240,5 +240,5 @@
       <inertia
         ixx="9.4187E-05"
-        ixy="1.2657E-19"
+        ixy="1.3079E-19"
         ixz="-1.4502E-16"
         iyy="4.476E-05"
@@ -290,5 +290,5 @@
     <inertial>
       <origin
-        xyz="0.028614 0.010457 -3.3307E-16"
+        xyz="0.028614 0.010457 -1.6653E-16"
         rpy="0 0 0" />
       <mass
@@ -299,5 +299,5 @@
         ixz="1.4501E-16"
         iyy="4.3878E-05"
-        iyz="-9.2657E-20"
+        iyz="-9.098E-20"
         izz="9.3658E-05" />
     </inertial>
@@ -347,15 +347,15 @@
     <inertial>
       <origin
-        xyz="-3.3307E-16 5.3794E-07 -0.0070001"
-        rpy="0 0 0" />
-      <mass
-        value="0.025977" />
-      <inertia
-        ixx="2.2053E-06"
-        ixy="8.338E-23"
-        ixz="-8.9123E-22"
-        iyy="2.2053E-06"
-        iyz="2.3258E-20"
-        izz="3.9777E-06" />
+        xyz="-4.44089209850063E-16 5.37938091368581E-07 -0.00700006055550945"
+        rpy="0 0 0" />
+      <mass
+        value="0.0259770442543706" />
+      <inertia
+        ixx="2.20534281951167E-06"
+        ixy="1.78671012311437E-22"
+        ixz="-8.79317315621994E-22"
+        iyy="2.20534281951168E-06"
+        iyz="2.32583060538047E-20"
+        izz="3.9777349014505E-06" />
     </inertial>
     <visual>
